File: pspac-astra-pmb.kicad_sch (KiCad schematic)
At the start: 11 parts, among them J1 Conn_01x02_Socket, J2 Conn_01x01_Socket, J3 Screw_Terminal_01x03, J4 Screw_Terminal_01x02, Q1 BSC014N04LSIATMA1, U1 INA226

Commit message: Add files via upload
Parts:
- removed J4: Screw_Terminal_01x02, TerminalBlock:TerminalBlock_bornier-2_P5.08mm, symbol Connector:Screw_Terminal_01x02
- added C2: 10u, symbol Device:C
- added C3: 100n, symbol Device:C
- added J5, J6: Screw_Terminal_01x01, symbol Connector:Screw_Terminal_01x01
- added U5: LD1117V33, Package_TO_SOT_THT:TO-220-3_Vertical, symbol Regulator_Linear:LD1117V33
Connections:
- net +12V: now also C3.1, J5.1 (Pin_1), U5.3 (VI)
- net GND: now also J3.1 (Pin_1), J3.2 (Pin_2), J3.3 (Pin_3), C2.2, C3.2, U5.1 (GND); no longer Q1.3 (S)
- net at R_shunt.4, U1.9 (Vin-): now also Q1.1 (D)
- net +3.3V: no longer names the net of C1.2, R2.1, R3.1, U1.6 (VS)
- net +3.3V: now also C2.1, U5.2 (VO)
- new net: J6.1 (Pin_1), Q1.3 (S)
Other:
- note added: "ESC"
- moved on the sheet: C1, J2, J3, Q1, R1

Commit message: Add files via upload
Parts:
- C1: footprint Capacitor_SMD:C_0805_2012Metric_Pad1.18x1.45mm_HandSolder -> (none)
- C3: footprint (none) -> Capacitor_SMD:C_1206_3216Metric_Pad1.33x1.80mm_HandSolder
- J1: footprint Connector_Wire:SolderWire-0.1sqmm_1x02_P3.6mm_D0.4mm_OD1mm -> Connector_PinSocket_2.00mm:PinSocket_1x02_P2.00mm_Vertical
- J2: footprint Connector_Wire:SolderWire-0.1sqmm_1x01_D0.4mm_OD1mm -> (none)
- R1, R2, R3: footprint Resistor_SMD:R_0805_2012Metric -> (none)
- R_shunt: value 1.4 mΩ -> 0.5 mΩ; footprint Resistor_SMD:R_Shunt_Vishay_WSK2512_6332Metric_T2.21mm -> (none)
Changed lines of the file:
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@@
 	)
 	(junction
-		(at 100.33 25.4)
+		(at 118.11 83.82)
+		(diameter 0)
+		(color 0 0 0 0)
+	)
+	(junction
+		(at 140.97 41.91)
+		(diameter 0)
+		(color 0 0 0 0)
+	)
+	(junction
+		(at 107.95 25.4)
+		(diameter 0)
+		(color 0 0 0 0)
+	)
+	(junction
+		(at 118.11 41.91)
+		(diameter 0)
+		(color 0 0 0 0)
+	)
+	(junction
+		(at 140.97 62.23)
+		(diameter 0)
+		(color 0 0 0 0)
+	)
+	(junction
+		(at 101.6 69.85)
+		(diameter 0)
+		(color 0 0 0 0)
+	)
+	(junction
+		(at 116.84 33.02)
+		(diameter 0)
+		(color 0 0 0 0)
+	)
+	(junction
+		(at 118.11 81.28)
+		(diameter 0)
+		(color 0 0 0 0)
+	)
+	(junction
+		(at 101.6 25.4)
+		(diameter 0)
+		(color 0 0 0 0)
+	)
+	(junction
+		(at 130.81 25.4)
+		(diameter 0)
+		(color 0 0 0 0)
+	)
+	(junction
+		(at 101.6 59.69)
 		(diameter 0)
 		(color 0 0 0 0)
@@
 	)
 	(junction
-		(at 140.97 41.91)
-		(diameter 0)
-		(color 0 0 0 0)
-	)
-	(junction
-		(at 107.95 25.4)
-		(diameter 0)
-		(color 0 0 0 0)
-	)
-	(junction
-		(at 118.11 41.91)
-		(diameter 0)
-		(color 0 0 0 0)
-	)
-	(junction
-		(at 140.97 62.23)
-		(diameter 0)
-		(color 0 0 0 0)
-	)
-	(junction
-		(at 101.6 69.85)
-		(diameter 0)
-		(color 0 0 0 0)
-	)
-	(junction
-		(at 118.11 81.28)
-		(diameter 0)
-		(color 0 0 0 0)
-	)
-	(junction
-		(at 116.84 33.02)
-		(diameter 0)
-		(color 0 0 0 0)
-	)
-	(junction
-		(at 130.81 25.4)
-		(diameter 0)
-		(color 0 0 0 0)
-	)
-	(junction
-		(at 101.6 59.69)
-		(diameter 0)
-		(color 0 0 0 0)
-	)
-	(junction
 		(at 121.92 33.02)
-		(diameter 0)
-		(color 0 0 0 0)
-	)
-	(junction
-		(at 118.11 83.82)
 		(diameter 0)
 		(color 0 0 0 0)
@@
 	(wire
 		(pts
-			(xy 100.33 25.4) (xy 100.33 59.69)
+			(xy 101.6 25.4) (xy 101.6 59.69)
+		)
+		(stroke
+			(width 0)
+			(type default)
+		)
+	)
+	(wire
+		(pts
+			(xy 101.6 25.4) (xy 107.95 25.4)
 		)
 		(stroke
@@
 	(wire
 		(pts
-			(xy 100.33 22.86) (xy 100.33 25.4)
+			(xy 101.6 20.32) (xy 101.6 25.4)
+		)
+		(stroke
+			(width 0)
+			(type default)
+		)
+	)
+	(wire
+		(pts
+			(xy 118.11 81.28) (xy 118.11 83.82)
 		)
 		(stroke
@@
 	(wire
 		(pts
-			(xy 118.11 81.28) (xy 118.11 83.82)
-		)
-		(stroke
-			(width 0)
-			(type default)
-		)
-	)
-	(wire
-		(pts
 			(xy 101.6 69.85) (xy 107.95 69.85)
 		)
@@
 	(wire
 		(pts
-			(xy 100.33 59.69) (xy 101.6 59.69)
-		)
-		(stroke
-			(width 0)
-			(type default)
-		)
-	)
-	(wire
-		(pts
 			(xy 132.08 41.91) (xy 140.97 41.91)
 		)
@@
 	(wire
 		(pts
+			(xy 118.11 83.82) (xy 118.11 86.36)
+		)
+		(stroke
+			(width 0)
+			(type default)
+		)
+	)
+	(wire
+		(pts
 			(xy 128.27 62.23) (xy 140.97 62.23)
 		)
@@
 	(wire
 		(pts
-			(xy 100.33 25.4) (xy 107.95 25.4)
-		)
-		(stroke
-			(width 0)
-			(type default)
-		)
-	)
-	(wire
-		(pts
-			(xy 118.11 83.82) (xy 118.11 86.36)
+			(xy 101.6 25.4) (xy 100.33 25.4)
 		)
 		(stroke
@@
 			)
 		)
-		(property "Footprint" "Connector_Wire:SolderWire-0.1sqmm_1x01_D0.4mm_OD1mm"
+		(property "Footprint" ""
 			(at 64.77 83.82 0)
 			(effects
@@
 			)
 		)
-		(property "Datasheet" "~"
+		(property "Datasheet" ""
 			(at 64.77 83.82 0)
 			(effects
@@
 			)
 		)
-		(property "Footprint" ""
+		(property "Footprint" "Capacitor_SMD:C_1206_3216Metric_Pad1.33x1.80mm_HandSolder"
 			(at 108.9152 33.02 0)
 			(effects
@@
 			)
 		)
-		(property "Description" "Unpolarized capacitor"
+		(property "Description" "81-GRM31CR72E104KW03"
 			(at 107.95 29.21 0)
 			(effects
@@
 			)
 		)
-		(property "Value" "1.4 mΩ"
+		(property "Value" "0.5 mΩ"
 			(at 99.06 66.0399 0)
 			(effects
@@
 			)
 		)
-		(property "Footprint" "Resistor_SMD:R_Shunt_Vishay_WSK2512_6332Metric_T2.21mm"
+		(property "Footprint" ""
 			(at 99.822 64.77 90)
 			(effects
@@
 			)
 		)
-		(property "Datasheet" "~"
+		(property "Datasheet" "https://fscdn.rohm.com/en/products/databook/datasheet/passive/resistor/chip_resistor/gmr-e.pdf"
 			(at 101.6 64.77 0)
 			(effects
@@
 	(symbol
 		(lib_id "power:+12V")
-		(at 100.33 22.86 0)
+		(at 101.6 20.32 0)
 		(unit 1)
 		(exclude_from_sim no)
@@
 		(dnp no)
 		(property "Reference" "#PWR01"
-			(at 100.33 26.67 0)
+			(at 101.6 24.13 0)
 			(effects
 				(font
@@
 		)
 		(property "Value" "+12V"
-			(at 96.266 21.844 0)
+			(at 97.536 19.304 0)
 			(effects
 				(font
@@
 		)
 		(property "Footprint" ""
-			(at 100.33 22.86 0)
+			(at 101.6 20.32 0)
 			(effects
 				(font
@@
 		)
 		(property "Datasheet" ""
-			(at 100.33 22.86 0)
+			(at 101.6 20.32 0)
 			(effects
 				(font
@@
 		)
 		(property "Description" "Power symbol creates a global label with name \"+12V\""
-			(at 100.33 22.86 0)
+			(at 101.6 20.32 0)
 			(effects
 				(font
@@
 		(on_board yes)
 		(dnp no)
-		(fields_autoplaced yes)
 		(property "Reference" "C1"
-			(at 109.22 34.29 90)
+			(at 106.172 40.132 90)
 			(effects
 				(font
@@
 		)
 		(property "Value" "0.1 u"
-			(at 109.22 36.83 90)
-			(effects
-				(font
-					(size 1.27 1.27)
-				)
-			)
-		)
-		(property "Footprint" "Capacitor_SMD:C_0805_2012Metric_Pad1.18x1.45mm_HandSolder"
+			(at 109.982 44.704 90)
+			(effects
+				(font
+					(size 1.27 1.27)
+				)
+			)
+		)
+		(property "Footprint" ""
 			(at 113.03 40.9448 0)
 			(effects
@@
 			)
 		)
-		(property "Datasheet" "~"
+		(property "Datasheet" "https://www.mouser.com/ProductDetail/Murata-Electronics/GRM188R71C104KA01D?qs=WZmVLWkT%2FeCcuvj%2FpnjfsA%3D%3D"
 			(at 109.22 41.91 0)
 			(effects
@@
 			)
 		)
-		(property "Footprint" "Resistor_SMD:R_0805_2012Metric"
+		(property "Footprint" ""
 			(at 130.302 52.07 90)
 			(effects
@@
 			)
 		)
-		(property "Datasheet" "~"
+		(property "Datasheet" "https://product.tdk.com/system/files/dam/doc/product/capacitor/ceramic/mlcc/catalog/mlcc_commercial_general_en.pdf"
 			(at 132.08 52.07 0)
 			(effects
@@
 		(on_board yes)
 		(dnp no)
-		(fields_autoplaced yes)
 		(property "Reference" "J3"
 			(at 125.73 82.5499 0)
@@
 			)
 		)
-		(property "Datasheet" "~"
+		(property "Datasheet" ""
 			(at 123.19 83.82 0)
 			(effects
@@
 			)
 		)
-		(property "Footprint" "Resistor_SMD:R_0805_2012Metric"
+		(property "Footprint" ""
 			(at 82.042 91.44 90)
 			(effects
@@
 			)
 		)
-		(property "Datasheet" "~"
+		(property "Datasheet" "https://www.mouser.com/ProductDetail/YAGEO/RC0603FR-0710KL?qs=grNVn54RoB%252B3GtjbJj3wJQ%3D%3D"
 			(at 83.82 91.44 0)
 			(effects
@@
 		(on_board yes)
 		(dnp no)
-		(fields_autoplaced yes)
 		(property "Reference" "J5"
 			(at 95.25 19.05 0)
@@
 		)
 		(property "Value" "Screw_Terminal_01x01"
-			(at 95.25 21.59 0)
+			(at 87.376 26.416 0)
 			(effects
 				(font
@@
 			)
 		)
-		(property "Datasheet" "~"
+		(property "Datasheet" ""
 			(at 95.25 25.4 0)
 			(effects
@@
 			)
 		)
-		(property "Footprint" "Resistor_SMD:R_0805_2012Metric"
+		(property "Footprint" ""
 			(at 139.192 52.07 90)
 			(effects
@@
 			)
 		)
-		(property "Datasheet" "~"
+		(property "Datasheet" "https://product.tdk.com/system/files/dam/doc/product/capacitor/ceramic/mlcc/catalog/mlcc_commercial_general_en.pdf"
 			(at 140.97 52.07 0)
 			(effects
@@
 			)
 		)
-		(property "Datasheet" "~"
+		(property "Datasheet" ""
 			(at 101.6 96.52 0)
 			(effects
@@
 			)
 		)
-		(property "Footprint" "Connector_Wire:SolderWire-0.1sqmm_1x02_P3.6mm_D0.4mm_OD1mm"
+		(property "Footprint" "Connector_PinSocket_2.00mm:PinSocket_1x02_P2.00mm_Vertical"
 			(at 161.29 62.23 0)
 			(effects
@@
 			)
 		)
-		(property "Datasheet" "~"
+		(property "Datasheet" ""
 			(at 161.29 62.23 0)
 			(effects

Commit message: Add files via upload
shunt resistor footprint added
Parts:
- removed R_shunt: 0.5 mΩ, symbol Device:R_Shunt
- added R_shunt: 0.5 mΩ, symbol Device:R
Connections:
- net +12V: now also R_shunt.1
- net at Q1.1 (D), U1.9 (Vin-): now also R_shunt.2
Changed lines of the file:
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@@
+	)
+	(junction
+		(at 101.6 59.69)
+		(diameter 0)
+		(color 0 0 0 0)
 	)
 	(junction
@@
 	)
 	(junction
+		(at 116.84 33.02)
+		(diameter 0)
+		(color 0 0 0 0)
+	)
+	(junction
+		(at 118.11 81.28)
+		(diameter 0)
+		(color 0 0 0 0)
+	)
+	(junction
+		(at 101.6 25.4)
+		(diameter 0)
+		(color 0 0 0 0)
+	)
+	(junction
+		(at 130.81 25.4)
+		(diameter 0)
+		(color 0 0 0 0)
+	)
+	(junction
+		(at 118.11 86.36)
+		(diameter 0)
+		(color 0 0 0 0)
+	)
+	(junction
+		(at 121.92 33.02)
+		(diameter 0)
+		(color 0 0 0 0)
+	)
+	(junction
+		(at 132.08 41.91)
+		(diameter 0)
+		(color 0 0 0 0)
+	)
+	(junction
+		(at 107.95 59.69)
+		(diameter 0)
+		(color 0 0 0 0)
+	)
+	(junction
+		(at 132.08 64.77)
+		(diameter 0)
+		(color 0 0 0 0)
+	)
+	(junction
 		(at 101.6 69.85)
 		(diameter 0)
@@
 	)
 	(junction
-		(at 116.84 33.02)
-		(diameter 0)
-		(color 0 0 0 0)
-	)
-	(junction
-		(at 118.11 81.28)
-		(diameter 0)
-		(color 0 0 0 0)
-	)
-	(junction
-		(at 101.6 25.4)
-		(diameter 0)
-		(color 0 0 0 0)
-	)
-	(junction
-		(at 130.81 25.4)
-		(diameter 0)
-		(color 0 0 0 0)
-	)
-	(junction
-		(at 101.6 59.69)
-		(diameter 0)
-		(color 0 0 0 0)
-	)
-	(junction
-		(at 118.11 86.36)
-		(diameter 0)
-		(color 0 0 0 0)
-	)
-	(junction
-		(at 121.92 33.02)
-		(diameter 0)
-		(color 0 0 0 0)
-	)
-	(junction
-		(at 132.08 41.91)
-		(diameter 0)
-		(color 0 0 0 0)
-	)
-	(junction
-		(at 107.95 59.69)
-		(diameter 0)
-		(color 0 0 0 0)
-	)
-	(junction
-		(at 132.08 64.77)
-		(diameter 0)
-		(color 0 0 0 0)
-	)
-	(junction
 		(at 83.82 83.82)
 		(diameter 0)
@@
 	(wire
 		(pts
-			(xy 101.6 67.31) (xy 101.6 69.85)
-		)
-		(stroke
-			(width 0)
-			(type default)
-		)
-	)
-	(wire
-		(pts
 			(xy 101.6 20.32) (xy 101.6 25.4)
 		)
@@
 	(wire
 		(pts
+			(xy 101.6 59.69) (xy 101.6 60.96)
+		)
+		(stroke
+			(width 0)
+			(type default)
+		)
+	)
+	(wire
+		(pts
 			(xy 130.81 25.4) (xy 140.97 25.4)
 		)
@@
 		(pts
 			(xy 107.95 33.02) (xy 116.84 33.02)
+		)
+		(stroke
+			(width 0)
+			(type default)
+		)
+	)
+	(wire
+		(pts
+			(xy 101.6 68.58) (xy 101.6 69.85)
 		)
 		(stroke
@@
 	)
 	(symbol
-		(lib_id "Device:R_Shunt")
+		(lib_id "Device:R")
 		(at 101.6 64.77 0)
 		(unit 1)
@@
 		(dnp no)
 		(property "Reference" "R_shunt"
-			(at 99.06 63.4999 0)
-			(effects
-				(font
-					(size 1.27 1.27)
-				)
-				(justify right)
+			(at 92.202 63.754 0)
+			(effects
+				(font
+					(size 1.27 1.27)
+				)
+				(justify left)
 			)
 		)
 		(property "Value" "0.5 mΩ"
-			(at 99.06 66.0399 0)
-			(effects
-				(font
-					(size 1.27 1.27)
-				)
-				(justify right)
+			(at 92.202 66.04 0)
+			(effects
+				(font
+					(size 1.27 1.27)
+				)
+				(justify left)
 			)
 		)
@@
 			)
 		)
-		(property "Datasheet" "https://fscdn.rohm.com/en/products/databook/datasheet/passive/resistor/chip_resistor/gmr-e.pdf"
+		(property "Datasheet" "~"
 			(at 101.6 64.77 0)
 			(effects
@@
 			)
 		)
-		(property "Description" "Shunt resistor with Kelvin connections"
+		(property "Description" "Resistor"
 			(at 101.6 64.77 0)
 			(effects
@@
 		(pin "1"
 		)
-		(pin "4"
-		)
 		(pin "2"
 		)
-		(pin "3"
-		)
 		(instances

Commit message: Add files via upload
Parts:
- removed R_shunt: 0.5 mΩ, symbol Device:R
- added R4: 0.5m, PSPAC:ShuntResistorPMB, symbol Device:R
- C1: footprint (none) -> Capacitor_SMD:C_0805_2012Metric_Pad1.18x1.45mm_HandSolder
- C3: footprint Capacitor_SMD:C_1206_3216Metric_Pad1.33x1.80mm_HandSolder -> (none)
- J1: footprint Connector_PinSocket_2.00mm:PinSocket_1x02_P2.00mm_Vertical -> Connector_Wire:SolderWire-0.1sqmm_1x02_P3.6mm_D0.4mm_OD1mm
- J2: footprint (none) -> Connector_Wire:SolderWire-0.1sqmm_1x01_D0.4mm_OD1mm
- R1, R2, R3: footprint (none) -> Resistor_SMD:R_0805_2012Metric
Connections:
- net +12V: now also R4.1
- net at Q1.1 (D), U1.9 (Vin-): now also R4.2
- no-connect marks 0 -> 3
