File: PSP_ASTRA_PMB.kicad_sch (KiCad schematic)
At the start: 15 parts, among them J1 Conn_01x02_Socket, J2 Conn_01x01_Socket, J3 Screw_Terminal_01x03, J5 Screw_Terminal_01x01, J6 Screw_Terminal_01x01, Q1 BSC014N04LSIATMA1, U1 INA226, U5 LD1117V33

Commit message: Add files via upload
Parts:
- Q1: footprint Package_TO_SOT_SMD:TDSON-8-1 -> PSPAC:MOSFETPMB
Connections:
- net Drain: now reaches Q1.1 (D), R4.2, U1.9 (Vin-)
- net Source: now reaches J6.1 (Pin_1), Q1.3 (S)

Commit message: Add files via upload
added pmos and voltage divider (see schematic)
Parts:
- added Q2: PMOS, PSPAC:PMOSPMB, symbol Simulation_SPICE:PMOS
- added R5: 10k, Resistor_SMD:R_0805_2012Metric_Pad1.20x1.40mm_HandSolder, symbol Device:R
- added R6: 10, Resistor_SMD:R_0805_2012Metric_Pad1.20x1.40mm_HandSolder, symbol Device:R
Connections:
- net +12V: now also R5.2
- net GND: now also Q1.3 (S)
- net Drain renamed PMOS Drain
- net PMOS Drain: now also Q2.1 (D); no longer Q1.1 (D)
- net Source renamed PMOS Source
- net PMOS Source: now also Q2.3 (S); no longer Q1.3 (S)
- new net NMOS Drain: Q1.1 (D), R6.1
- new net PMOS Gate: Q2.2 (G), R5.1, R6.2
Other:
- moved on the sheet: J2, Q1, R1

Commit message: Add files via upload
Parts:
- C1: Purchase Links (none) -> https://www.digikey.com/en/products/detail/yageo/AC0805KFX7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
- C2: Purchase Links (none) -> https://www.digikey.com/en/products/detail/samsung-electro-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
- C3: value 100n -> 0.1 u; Purchase Links (none) -> https://www.digikey.com/en/products/detail/yageo/AC0805KFX7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
- J3: Purchase Links (none) -> https://www.mouser.com/ProductDetail/Altech/MV-1003?qs=sGAE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
- J5, J6: Purchase Links (none) -> https://www.mouser.com/ProductDetail/Altech/MV-1001?qs=vvQt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
- Q1: Purchase Links (none) -> https://www.digikey.com/en/products/detail/infineon-technol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
- Q2: Purchase Links (none) -> https://www.digikey.com/en/products/detail/vishay-siliconix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
- R1, R5: Purchase Links (none) -> https://www.digikey.com/en/products/detail/yageo/AT0805BRD0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
- R2, R3: Purchase Links (none) -> https://www.digikey.com/en/products/detail/vishay-dale/CRCW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
- R4: Purchase Links (none) -> https://www.digikey.com/en/products/detail/rohm-semiconduct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
- R6: Purchase Links (none) -> https://www.digikey.com/en/products/detail/yageo/RC0805DR-0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
- U1: Purchase Links (none) -> https://www.digikey.com/en/products/detail/texas-instrument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
- U5: Purchase Links (none) -> https://www.digikey.com/en/products/detail/stmicroelectroni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
Changed lines of the file:
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@@
+			)
+		)
+		(property "Purchase Links" "https://www.digikey.com/en/products/detail/vishay-siliconix/SI7141DP-T1-GE3/2441718"
+			(at 125.73 115.57 0)
+			(effects
+				(font
+					(size 1.27 1.27)
+				)
+				(hide yes)
 			)
 		)
@@
 			)
 		)
-		(property "Purchase Links" ""
+		(property "Purchase Links" "https://www.digikey.com/en/products/detail/samsung-electro-mechanics/CL31B106KAHNNNE/3887462"
 			(at 157.48 66.04 0)
 			(effects
@@
 			)
 		)
-		(property "Purchase Links" ""
+		(property "Purchase Links" "https://www.digikey.com/en/products/detail/rohm-semiconductor/PSR500HTQFF0L50/4864193"
 			(at 128.27 101.6 0)
 			(effects
@@
 			)
 		)
+		(property "Purchase Links" "https://www.digikey.com/en/products/detail/yageo/RC0805DR-0710RL/21767346"
+			(at 113.03 115.57 90)
+			(effects
+				(font
+					(size 1.27 1.27)
+				)
+				(hide yes)
+			)
+		)
 		(pin "2"
 		)
@@
 			)
 		)
-		(property "Purchase Links" ""
+		(property "Purchase Links" "https://www.digikey.com/en/products/detail/stmicroelectronics/LD1117V33/586012"
 			(at 148.59 62.23 0)
 			(effects
@@
 			)
 		)
-		(property "Purchase Links" ""
+		(property "Purchase Links" "https://www.digikey.com/en/products/detail/texas-instruments/INA226AIDGSR/2687236"
 			(at 144.78 99.06 0)
 			(effects
@@
 			)
 		)
-		(property "Value" "100n"
+		(property "Value" "0.1 u"
 			(at 137.414 67.31 0)
 			(effects
@@
 			)
 		)
-		(property "Purchase Links" ""
+		(property "Purchase Links" "https://www.digikey.com/en/products/detail/yageo/AC0805KFX7R9BB104/18106225"
 			(at 134.62 66.04 0)
 			(effects
@@
 		)
 		(property "Description" "Resistor"
+			(at 120.65 106.68 0)
+			(effects
+				(font
+					(size 1.27 1.27)
+				)
+				(hide yes)
+			)
+		)
+		(property "Purchase Links" "https://www.digikey.com/en/products/detail/yageo/AT0805BRD0710KL/5139579"
 			(at 120.65 106.68 0)
 			(effects
@@
 			)
 		)
-		(property "Purchase Links" ""
+		(property "Purchase Links" "https://www.digikey.com/en/products/detail/yageo/AC0805KFX7R9BB104/18106225"
 			(at 135.89 78.74 90)
 			(effects
@@
 			)
 		)
-		(property "Purchase Links" ""
+		(property "Purchase Links" "https://www.digikey.com/en/products/detail/vishay-dale/CRCW08054K70FKEA/1175713"
 			(at 158.75 88.9 0)
 			(effects
@@
 			)
 		)
-		(property "Purchase Links" ""
+		(property "Purchase Links" "https://www.digikey.com/en/products/detail/infineon-technologies/BSC014N04LSIATMA1/4318669?gclsrc=aw.ds&gad_source=1&gad_campaignid=120565755&gbraid=0AAAAADrbLlhCXftiJluGgUch6rsfE1-Oc&gclid=Cj0KCQjw35bIBhDqARIsAGjd-cbBiOx49j1MpeQSxlyjZuZO4I6EF-hOGT98txcq7WNj8aYbzVh5hE4aAsg7EALw_wcB"
 			(at 102.87 120.65 0)
 			(effects
@@
 			)
 		)
-		(property "Purchase Links" ""
+		(property "Purchase Links" "https://www.mouser.com/ProductDetail/Altech/MV-1003?qs=sGAEpiMZZMvPvGwLNS6718Cc%252BAzGpzUtSDuHJgDMGAE%3D"
 			(at 149.86 120.65 0)
 			(effects
@@
 			)
 		)
-		(property "Purchase Links" ""
+		(property "Purchase Links" "https://www.digikey.com/en/products/detail/yageo/AT0805BRD0710KL/5139579"
 			(at 93.98 128.27 0)
 			(effects
@@
 			)
 		)
-		(property "Purchase Links" ""
+		(property "Purchase Links" "https://www.mouser.com/ProductDetail/Altech/MV-1001?qs=vvQtp7zwQdOvsbaLONf9Bw%3D%3D"
 			(at 121.92 62.23 0)
 			(effects
@@
 			)
 		)
-		(property "Purchase Links" ""
+		(property "Purchase Links" "https://www.digikey.com/en/products/detail/vishay-dale/CRCW08054K70FKEA/1175713"
 			(at 167.64 88.9 0)
 			(effects
@@
 			)
 		)
-		(property "Purchase Links" ""
+		(property "Purchase Links" "https://www.mouser.com/ProductDetail/Altech/MV-1001?qs=vvQtp7zwQdOvsbaLONf9Bw%3D%3D"
 			(at 128.27 133.35 90)
 			(effects

Commit message: Add files via upload
Parts:
- added H1, H2, H3, H4: MountingHole, MountingHole:MountingHole_3.2mm_M3, symbol Mechanical:MountingHole
- C2: Purchase Links https://www.digikey.com/en/products/detail/samsung-electro-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 -> https://www.digikey.com/en/products/detail/yageo/CC0805KKX5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
Connections:
- net PMOS Drain: now also J6.1 (Pin_1); no longer R4.2, U1.9 (Vin-)
- net PMOS Source: now also R4.2, U1.9 (Vin-); no longer J6.1 (Pin_1)
